File: Eagle Files/BMXBreakoutTiny/BMX055.sch (EAGLE design)
At the start: 5 parts, among them U1 BMX055

Commit message: Forgot to add the dimension
Parts:
- removed FRAME1: FRAME-LETTER, SparkFun-Aesthetics:FRAME-LETTER
Changed lines of the file:
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@@
 </classes>
 <parts>
-<part name="FRAME1" library="SparkFun-Aesthetics" deviceset="FRAME-LETTER" device=""/>
 <part name="U1" library="x-io" deviceset="BMX055" device=""/>
 <part name="GND2" library="SparkFun-Aesthetics" deviceset="GND" device=""/>
@@
 </plain>
 <instances>
-<instance part="FRAME1" gate="G$1" x="0" y="0"/>
-<instance part="FRAME1" gate="G$2" x="147.32" y="0"/>
 <instance part="U1" gate="G$1" x="114.3" y="114.3"/>
 <instance part="GND2" gate="1" x="142.24" y="111.76" rot="R90"/>
